File: kicad/stoper.kicad_pcb (KiCad board)
At the start: 2 copper layers, 29 parts

Commit message: finish designing pcb
Parts:
- added REF1: MountingHole_2.2mm_M2, MountingHole:MountingHole_2.2mm_M2, F.Cu at (74.9, 49.5)
- added REF2: MountingHole_2.2mm_M2, MountingHole:MountingHole_2.2mm_M2, F.Cu at (172.7, 49.5)
- added REF3: MountingHole_2.2mm_M2, MountingHole:MountingHole_2.2mm_M2, F.Cu at (74.9, 125.7)
- added REF4: MountingHole_2.2mm_M2, MountingHole:MountingHole_2.2mm_M2, F.Cu at (172.7, 125.7)
- moved R11 48.4 mm to (130.8, 67.3)
- moved R9 37.0 mm to (123.2, 67.3)
- moved DefaultOff1 33.8 mm to (108.7, 120.7)
- moved PWR1 32.5 mm to (87.6, 104.8)
- moved R2 26.2 mm to (94.0, 116.8)
- moved R6 22.2 mm to (108.0, 57.1)
- moved R1 19.3 mm to (78.7, 116.8)
- moved R3 16.9 mm to (92.7, 87.6), turned to 90 degrees
- moved R8 9.78 mm to (115.6, 57.1), turned to -90 degrees
- moved C1 7.27 mm to (92.7, 69.6)
- moved OnOffLed1 5.48 mm to (91.6, 95.1)
- moved MillisecondsTimer1 5.24 mm to (77.5, 71.1)
- moved OnOff1 5.22 mm to (77.5, 86.4)
- moved DefaultReset1 3.81 mm to (129.5, 120.7)
- moved SingleSecondsCounter1 1.27 mm to (152.4, 78.8)
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Routing:
- net GND: track 0.00 -> 474.9 mm
- net /+9V: track 0.00 -> 266.9 mm
- net /MilliSecondsPulse1: track 0.00 -> 159.2 mm
- net /ResetButtonIn1: track 0.00 -> 133.6 mm
- net /SingleSecondsPulse1: track 0.00 -> 111.6 mm
- net Net-(R8-Pad1): track 0.00 -> 110.2 mm
- net Net-(On1-Pad1): track 0.00 -> 105.1 mm
- net Net-(DefaultOff1-Pad2): track 0.00 -> 104.2 mm
- net /TimerPower1: track 0.00 -> 95.1 mm
- net Net-(DoubleSecondsCounter1-Pad10): track 0.00 -> 88.9 mm
- net Net-(MilliSecondsCounter1-Pad10): track 0.00 -> 82.4 mm
- net /DoubleSecondsPulse1: track 0.00 -> 81.3 mm
- net Net-(DoubleSecondsCounter1-Pad11): track 0.00 -> 77.8 mm
- net Net-(DoubleSecondsCounter1-Pad12): track 0.00 -> 76.9 mm
- net Net-(DoubleSecondsCounter1-Pad6): track 0.00 -> 70.8 mm
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Other:
- board outline added: 105.4 x 83.8 mm
